File: schematics/tube-board/vumeter-schematics.kicad_pcb (KiCad board)
At the start: 2 copper layers, 100 x 30 mm, 51 parts, among them J1 SWD, J2 Conn_01x04, J3 Conn_01x04, J4 Standoff_1, J5 Standoff_2, J6 Conn_01x01_Male, J7 Conn_01x01_Male, Q1 MJE340, Q2 MJE340, Q3 MJE340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

Commit message: ok
Other:
- net class 75V removed
- net class Default removed
- net class HV removed
